File: hardware/Looper.sch (KiCad schematic (older format))
At the start: 1 part

Commit message: Replace Sig-GND label by global GNDA label
Connections:
- net Sig-GND renamed GNDA
Changed lines of the file:
@@
 $Descr A4 11693 8268
 encoding utf-8
-Sheet 5 19
+Sheet 7 19
 Title ""
 Date ""
@@
 F5 "FX_Return" I R 4500 3500 60
 F6 "9V" I L 3400 4000 60
-F7 "Sig-GND" I L 3400 4200 60
-F8 "Ctrl" I L 3400 4400 60
+F7 "Ctrl" I L 3400 4400 60
 $EndSheet
 $Comp
@@
 AR Path="/54D120FF/54E9BE87/54E9CF0E" Ref="CON?"  Part="1"
 AR Path="/54D120FF/54EA08CB/54E9CF0E" Ref="CON?"  Part="1"
+AR Path="/54D120FF/54E9F8A8/54E9CF0E" Ref="CON?"  Part="1"
 F 0 "CON?" H 5900 5250 60  0000 C CNN
 F 1 "Jack_Stacked" H 5850 3500 60  0000 C CNN
@@
 	4700 1450 5300 1450
 Wire Wire Line
-	5300 3200 3200 3200
-Wire Wire Line
-	3200 3200 3200 4200
-Wire Wire Line
-	2800 4200 3400 4200
-Wire Wire Line
-	5100 1550 5100 3200
+	5100 1550 5100 3300
 Wire Wire Line
 	5100 1650 5300 1650
@@
 Wire Wire Line
 	4500 3700 5300 3700
-Text HLabel 2800 4200 0    60   Input ~ 0
-Sig-GND
-Connection ~ 3200 4200
+$Comp
+L GNDA #PWR?
+U 1 1 54EA1A07
+P 5100 3300
+AR Path="/54D120FF/54E9F8A8/54EA1A07" Ref="#PWR?"  Part="1"
+AR Path="/54D120FF/54E9BE87/54EA1A07" Ref="#PWR?"  Part="1"
+F 0 "#PWR?" H 5100 3050 60  0001 C CNN
+F 1 "GNDA" H 5100 3150 60  0000 C CNN
+F 2 "" H 5100 3300 60  0000 C CNN
+F 3 "" H 5100 3300 60  0000 C CNN
+	1    5100 3300
+	1    0    0    -1
+$EndComp
+Wire Wire Line
+	5100 3200 5300 3200
 $EndSCHEMATC

Commit message: Use global label for digital (noisy) 9V
Changed lines of the file:
@@
 F4 "FX_Send" O L 3400 3500 60
 F5 "FX_Return" I R 4500 3500 60
-F6 "9V" I L 3400 4000 60
 F7 "Ctrl" I L 3400 4400 60
 $EndSheet
@@
 	5300 1550 5100 1550
 Connection ~ 5100 1650
-Text HLabel 2800 4000 0    60   Input ~ 0
-9V
 Text HLabel 2800 4400 0    60   Input ~ 0
 Ctrl
@@
 	2800 3700 3400 3700
 Wire Wire Line
-	2800 4000 3400 4000
-Wire Wire Line
 	2800 4400 3400 4400

Commit message: Draw looper chain
Other:
- note added: "FX Return"
- note added: "FX Send"
Changed lines of the file:
@@
 $Descr A4 11693 8268
 encoding utf-8
-Sheet 7 19
+Sheet 15 19
 Title ""
 Date ""
@@
 $EndDescr
 $Sheet
-S 3400 3400 1100 1100
+S 3400 3400 1100 600
 U 54E9BE9F
 F0 "Single True Bypass" 60
@@
 F4 "FX_Send" O L 3400 3500 60
 F5 "FX_Return" I R 4500 3500 60
-F7 "Ctrl" I L 3400 4400 60
+F6 "Ctrl" I L 3400 3900 60
 $EndSheet
 $Comp
@@
 	5300 1550 5100 1550
 Connection ~ 5100 1650
-Text HLabel 2800 4400 0    60   Input ~ 0
+Text HLabel 2800 3900 0    60   Input ~ 0
 Ctrl
 Text HLabel 2800 3700 0    60   Input ~ 0
@@
 Wire Wire Line
 	2800 3700 3400 3700
-Wire Wire Line
-	2800 4400 3400 4400
 Wire Wire Line
 	4500 3700 5300 3700
@@
 Wire Wire Line
 	5100 3200 5300 3200
+Text Notes 6850 2950 0    60   ~ 0
+FX Send
+Text Notes 6850 2100 0    60   ~ 0
+FX Return
+Wire Wire Line
+	2800 3900 3400 3900
 $EndSCHEMATC
