File: hardware/looper.sch (KiCad schematic (older format))
At the start: 1 part

Commit message: Assign project specific footprints
Parts:
- CON?: footprint (none) -> uMIDI-FX:NSJ12HF-1
Changed lines of the file:
@@
 $Descr A4 11693 8268
 encoding utf-8
-Sheet 10 21
+Sheet 18 21
 Title ""
 Date ""
@@
 F 0 "CON?" H 5900 5250 60  0000 C CNN
 F 1 "Jack_Stacked" H 5850 3500 60  0000 C CNN
-F 2 "" H 6750 3250 60  0000 C CNN
+F 2 "uMIDI-FX:NSJ12HF-1" H 6750 3250 60  0001 C CNN
 F 3 "" H 6750 3250 60  0000 C CNN
 	1    6750 3250

Commit message: Annotate schematic components
Parts:
- gave numbers to parts that had none: 1
Changed lines of the file:
@@
 $Descr A4 11693 8268
 encoding utf-8
-Sheet 18 21
+Sheet 14 21
 Title ""
 Date ""
@@
 $EndSheet
 $Comp
-L Jack_Stacked CON?
+L Jack_Stacked CON17
 U 1 1 54E9CF0E
 P 6750 3250
-AR Path="/54D120FF/54E9BE87/54E9CF0E" Ref="CON?"  Part="1"
-AR Path="/54D120FF/54EA08CB/54E9CF0E" Ref="CON?"  Part="1"
-AR Path="/54D120FF/54E9F8A8/54E9CF0E" Ref="CON?"  Part="1"
-AR Path="/54D120FF/54E9FD8E/54E9CF0E" Ref="CON?"  Part="1"
-AR Path="/54D120FF/54EA08BF/54E9CF0E" Ref="CON?"  Part="1"
-AR Path="/54D120FF/54EA08C5/54E9CF0E" Ref="CON?"  Part="1"
-F 0 "CON?" H 5900 5250 60  0000 C CNN
+AR Path="/54D120FF/54E9BE87/54E9CF0E" Ref="CON17"  Part="1"
+AR Path="/54D120FF/54EA08CB/54E9CF0E" Ref="CON16"  Part="1"
+AR Path="/54D120FF/54E9F8A8/54E9CF0E" Ref="CON12"  Part="1"
+AR Path="/54D120FF/54E9FD8E/54E9CF0E" Ref="CON13"  Part="1"
+AR Path="/54D120FF/54EA08BF/54E9CF0E" Ref="CON14"  Part="1"
+AR Path="/54D120FF/54EA08C5/54E9CF0E" Ref="CON15"  Part="1"
+F 0 "CON15" H 5900 5250 60  0000 C CNN
 F 1 "Jack_Stacked" H 5850 3500 60  0000 C CNN
 F 2 "uMIDI-FX:NSJ12HF-1" H 6750 3250 60  0001 C CNN
@@
 	4500 3700 5300 3700
 $Comp
-L GNDA #PWR?
+L GNDA #PWR88
 U 1 1 54EA1A07
 P 5100 3300
-AR Path="/54D120FF/54E9F8A8/54EA1A07" Ref="#PWR?"  Part="1"
-AR Path="/54D120FF/54E9BE87/54EA1A07" Ref="#PWR?"  Part="1"
-AR Path="/54D120FF/54E9FD8E/54EA1A07" Ref="#PWR?"  Part="1"
-AR Path="/54D120FF/54EA08BF/54EA1A07" Ref="#PWR?"  Part="1"
-AR Path="/54D120FF/54EA08C5/54EA1A07" Ref="#PWR?"  Part="1"
-AR Path="/54D120FF/54EA08CB/54EA1A07" Ref="#PWR?"  Part="1"
-F 0 "#PWR?" H 5100 3050 60  0001 C CNN
+AR Path="/54D120FF/54E9F8A8/54EA1A07" Ref="#PWR88"  Part="1"
+AR Path="/54D120FF/54E9BE87/54EA1A07" Ref="#PWR123"  Part="1"
+AR Path="/54D120FF/54E9FD8E/54EA1A07" Ref="#PWR95"  Part="1"
+AR Path="/54D120FF/54EA08BF/54EA1A07" Ref="#PWR102"  Part="1"
+AR Path="/54D120FF/54EA08C5/54EA1A07" Ref="#PWR109"  Part="1"
+AR Path="/54D120FF/54EA08CB/54EA1A07" Ref="#PWR116"  Part="1"
+F 0 "#PWR109" H 5100 3050 60  0001 C CNN
 F 1 "GNDA" H 5100 3150 60  0000 C CNN
 F 2 "" H 5100 3300 60  0000 C CNN

Commit message: Replace barrel jack symbols
Changed lines of the file:
@@
 $Descr A4 11693 8268
 encoding utf-8
-Sheet 14 21
+Sheet 12 21
 Title ""
 Date ""
@@
 AR Path="/54D120FF/54EA08BF/54E9CF0E" Ref="CON14"  Part="1"
 AR Path="/54D120FF/54EA08C5/54E9CF0E" Ref="CON15"  Part="1"
-F 0 "CON15" H 5900 5250 60  0000 C CNN
+F 0 "CON14" H 5900 5250 60  0000 C CNN
 F 1 "Jack_Stacked" H 5850 3500 60  0000 C CNN
 F 2 "uMIDI-FX:NSJ12HF-1" H 6750 3250 60  0001 C CNN
@@
 AR Path="/54D120FF/54EA08C5/54EA1A07" Ref="#PWR109"  Part="1"
 AR Path="/54D120FF/54EA08CB/54EA1A07" Ref="#PWR116"  Part="1"
-F 0 "#PWR109" H 5100 3050 60  0001 C CNN
+F 0 "#PWR102" H 5100 3050 60  0001 C CNN
 F 1 "GNDA" H 5100 3150 60  0000 C CNN
 F 2 "" H 5100 3300 60  0000 C CNN
