File: hardware/loopers.sch (KiCad schematic (older format))
At the start: 2 parts

Commit message: Assign project specific footprints
Parts:
- CON? (x2): footprint (none) -> uMIDI-FX:NSJ12HF-1
Changed lines of the file:
@@
 F 0 "CON?" H 2300 4550 60  0000 C CNN
 F 1 "Jack_Stacked" H 2250 2800 60  0000 C CNN
-F 2 "" H 3150 2550 60  0000 C CNN
+F 2 "uMIDI-FX:NSJ12HF-1" H 3150 2550 60  0001 C CNN
 F 3 "" H 3150 2550 60  0000 C CNN
 	1    3150 2550
@@
 F 0 "CON?" H 7500 4550 60  0000 C CNN
 F 1 "Jack_Stacked" H 7450 2800 60  0000 C CNN
-F 2 "" H 8350 2550 60  0000 C CNN
+F 2 "uMIDI-FX:NSJ12HF-1" H 8350 2550 60  0001 C CNN
 F 3 "" H 8350 2550 60  0000 C CNN
 	1    8350 2550

Commit message: Annotate schematic components
Parts:
- gave numbers to parts that had none: 2
Changed lines of the file:
@@
 $EndSheet
 $Comp
-L Jack_Stacked CON?
+L Jack_Stacked CON10
 U 1 1 54E9736C
 P 3150 2550
-F 0 "CON?" H 2300 4550 60  0000 C CNN
+F 0 "CON10" H 2300 4550 60  0000 C CNN
 F 1 "Jack_Stacked" H 2250 2800 60  0000 C CNN
 F 2 "uMIDI-FX:NSJ12HF-1" H 3150 2550 60  0001 C CNN
@@
 	1200 2000 1700 2000
 $Comp
-L GNDA #PWR?
+L GNDA #PWR79
 U 1 1 54E9875E
 P 2500 3000
-F 0 "#PWR?" H 2500 2750 60  0001 C CNN
+F 0 "#PWR79" H 2500 2750 60  0001 C CNN
 F 1 "GNDA" H 2500 2850 60  0000 C CNN
 F 2 "" H 2500 3000 60  0000 C CNN
@@
 	2500 3200 2400 3200
 $Comp
-L GNDA #PWR?
+L GNDA #PWR78
 U 1 1 54E98AC8
 P 1600 2600
-F 0 "#PWR?" H 1600 2350 60  0001 C CNN
+F 0 "#PWR78" H 1600 2350 60  0001 C CNN
 F 1 "GNDA" H 1600 2450 60  0000 C CNN
 F 2 "" H 1600 2600 60  0000 C CNN
@@
 Connection ~ 1600 1900
 $Comp
-L Jack_Stacked CON?
+L Jack_Stacked CON11
 U 1 1 54E99C5E
 P 8350 2550
-F 0 "CON?" H 7500 4550 60  0000 C CNN
+F 0 "CON11" H 7500 4550 60  0000 C CNN
 F 1 "Jack_Stacked" H 7450 2800 60  0000 C CNN
 F 2 "uMIDI-FX:NSJ12HF-1" H 8350 2550 60  0001 C CNN
@@
 $EndComp
 $Comp
-L GNDA #PWR?
+L GNDA #PWR81
 U 1 1 54E9A297
 P 9900 2600
-F 0 "#PWR?" H 9900 2350 60  0001 C CNN
+F 0 "#PWR81" H 9900 2350 60  0001 C CNN
 F 1 "GNDA" H 9900 2450 60  0000 C CNN
 F 2 "" H 9900 2600 60  0000 C CNN
@@
 	10100 1150 9800 1150
 $Comp
-L GNDA #PWR?
+L GNDA #PWR80
 U 1 1 54E9B679
 P 9900 1350
-F 0 "#PWR?" H 9900 1100 60  0001 C CNN
+F 0 "#PWR80" H 9900 1100 60  0001 C CNN
 F 1 "GNDA" H 9900 1200 60  0000 C CNN
 F 2 "" H 9900 1350 60  0000 C CNN
