File: hardware/power.sch (KiCad schematic (older format))
At the start: 62 parts

Commit message: Annotate schematic components
Parts:
- gave numbers to parts that had none: 62

Commit message: Replace barrel jack symbols
Parts:
- removed CON1: 12V in, symbol BARREL_JACK
- removed CON2, CON3, CON4, CON5, CON6, CON7, CON8: 9V out, symbol BARREL_JACK
- added P?: 9V out A, Connect:PINHEAD1-2, symbol CONN_01X02
- added P?: 9V out B, Connect:PINHEAD1-2, symbol CONN_01X02
- added P?: 9V out C, Connect:PINHEAD1-2, symbol CONN_01X02
- added P?: 12V in, Connect:PINHEAD1-2, symbol CONN_01X02
Connections:
- wire segments 110 -> 95
Other:
- moved on the sheet: C29, C30, C32, C33, C35, C36, C38, C39, U8, U9

Commit message: Add global 5V rail
Parts:
- added C? (x2): 100n, symbol C
- added C? (x2): 10u, symbol C
- added U?: LM7805CT, TO-220, symbol LM7805CT
Connections:
- net +12V: now also C?.1, C?.1, U?.1 (IN)
- net GND: now also C?.2, C?.2, C?.2, C?.2, U?.2 (GND)
- new net +5V: C?.1, C?.1, U?.3 (OUT)
Other:
- note added: "Global digital 5V"
- note added: "Global digital 9V"
- note removed: "Global digital 9V for uMidi and loopers"
Changed lines of the file:
@@
 Wire Wire Line
 	3050 5300 3050 5250
-Text Notes 1300 5000 0    60   ~ 0
-Global digital 9V for uMidi and loopers
+Text Notes 2650 5000 0    60   ~ 0
+Global digital 9V
 $Comp
 L GND #PWR57
@@
 Wire Wire Line
 	1500 1200 1400 1200
+$Comp
+L C C?
+U 1 1 54E9F4F7
+P 1450 6850
+F 0 "C?" H 1500 6950 50  0000 L CNN
+F 1 "100n" H 1500 6750 50  0000 L CNN
+F 2 "" H 1488 6700 30  0000 C CNN
+F 3 "" H 1450 6850 60  0000 C CNN
+	1    1450 6850
+	1    0    0    -1
+$EndComp
+$Comp
+L C C?
+U 1 1 54E9F4FD
+P 2450 6850
+F 0 "C?" H 2500 6950 50  0000 L CNN
+F 1 "100n" H 2500 6750 50  0000 L CNN
+F 2 "" H 2488 6700 30  0000 C CNN
+F 3 "" H 2450 6850 60  0000 C CNN
+	1    2450 6850
+	1    0    0    -1
+$EndComp
+$Comp
+L +12V #PWR?
+U 1 1 54E9F503
+P 1150 6450
+F 0 "#PWR?" H 1150 6300 60  0001 C CNN
+F 1 "+12V" H 1150 6590 60  0000 C CNN
+F 2 "" H 1150 6450 60  0000 C CNN
+F 3 "" H 1150 6450 60  0000 C CNN
+	1    1150 6450
+	1    0    0    -1
+$EndComp
+$Comp
+L GND #PWR?
+U 1 1 54E9F509
+P 1150 7050
+F 0 "#PWR?" H 1150 6800 60  0001 C CNN
+F 1 "GND" H 1150 6900 60  0000 C CNN
+F 2 "" H 1150 7050 60  0000 C CNN
+F 3 "" H 1150 7050 60  0000 C CNN
+	1    1150 7050
+	1    0    0    -1
+$EndComp
+$Comp
+L GND #PWR?
+U 1 1 54E9F50F
+P 1450 7050
+F 0 "#PWR?" H 1450 6800 60  0001 C CNN
+F 1 "GND" H 1450 6900 60  0000 C CNN
+F 2 "" H 1450 7050 60  0000 C CNN
+F 3 "" H 1450 7050 60  0000 C CNN
+	1    1450 7050
+	1    0    0    -1
+$EndComp
+$Comp
+L GND #PWR?
+U 1 1 54E9F515
+P 2450 7050
+F 0 "#PWR?" H 2450 6800 60  0001 C CNN
+F 1 "GND" H 2450 6900 60  0000 C CNN
+F 2 "" H 2450 7050 60  0000 C CNN
+F 3 "" H 2450 7050 60  0000 C CNN
+	1    2450 7050
+	1    0    0    -1
+$EndComp
+$Comp
+L GND #PWR?
+U 1 1 54E9F51B
+P 2750 7050
+F 0 "#PWR?" H 2750 6800 60  0001 C CNN
+F 1 "GND" H 2750 6900 60  0000 C CNN
+F 2 "" H 2750 7050 60  0000 C CNN
+F 3 "" H 2750 7050 60  0000 C CNN
+	1    2750 7050
+	1    0    0    -1
+$EndComp
+$Comp
+L GND #PWR?
+U 1 1 54E9F521
+P 1950 7050
+F 0 "#PWR?" H 1950 6800 60  0001 C CNN
+F 1 "GND" H 1950 6900 60  0000 C CNN
+F 2 "" H 1950 7050 60  0000 C CNN
+F 3 "" H 1950 7050 60  0000 C CNN
+	1    1950 7050
+	1    0    0    -1
+$EndComp
+$Comp
+L C C?
+U 1 1 54E9F527
+P 1150 6850
+F 0 "C?" H 1200 6950 50  0000 L CNN
+F 1 "10u" H 1200 6750 50  0000 L CNN
+F 2 "" H 1188 6700 30  0000 C CNN
+F 3 "" H 1150 6850 60  0000 C CNN
+	1    1150 6850
+	1    0    0    -1
+$EndComp
+$Comp
+L C C?
+U 1 1 54E9F52D
+P 2750 6850
+F 0 "C?" H 2800 6950 50  0000 L CNN
+F 1 "10u" H 2800 6750 50  0000 L CNN
+F 2 "" H 2788 6700 30  0000 C CNN
+F 3 "" H 2750 6850 60  0000 C CNN
+	1    2750 6850
+	1    0    0    -1
+$EndComp
+Wire Wire Line
+	1150 6550 1550 6550
+Wire Wire Line
+	1150 6450 1150 6650
+Wire Wire Line
+	1450 6650 1450 6550
+Connection ~ 1450 6550
+Wire Wire Line
+	2750 6550 2750 6650
+Wire Wire Line
+	2450 6650 2450 6550
+Connection ~ 2450 6550
+Connection ~ 2750 6550
+Connection ~ 1150 6550
+Wire Wire Line
+	1950 7050 1950 6850
+Wire Wire Line
+	2350 6550 3050 6550
+Wire Wire Line
+	3050 6550 3050 6500
+Text Notes 2650 6300 0    60   ~ 0
+Global digital 5V
+$Comp
+L LM7805CT U?
+U 1 1 54EA0421
+P 1950 6600
+F 0 "U?" H 1750 6800 40  0000 C CNN
+F 1 "LM7805CT" H 1950 6800 40  0000 L CNN
+F 2 "TO-220" H 1950 6700 30  0000 C CIN
+F 3 "" H 1950 6600 60  0000 C CNN
+	1    1950 6600
+	1    0    0    -1
+$EndComp
+$Comp
+L +5V #PWR?
+U 1 1 54EA0563
+P 3050 6500
+F 0 "#PWR?" H 3050 6350 60  0001 C CNN
+F 1 "+5V" H 3050 6640 60  0000 C CNN
+F 2 "" H 3050 6500 60  0000 C CNN
+F 3 "" H 3050 6500 60  0000 C CNN
+	1    3050 6500
+	1    0    0    -1
+$EndComp
 $EndSCHEMATC
