File: hardware/switch.sch (KiCad schematic (older format))
At the start: 6 parts

Commit message: Add switcher relais
Parts:
- added REL?: Meder SIL05-1A72-71L, symbol Relais_SPST
- added REL?: Relais_SPST, symbol Relais_SPST
Connections:
- wire segments 18 -> 20
Other:
- note removed: "TODO"
Changed lines of the file:
@@
 $Descr A4 11693 8268
 encoding utf-8
-Sheet 17 21
+Sheet 20 21
 Title ""
 Date ""
@@
 Text HLabel 4900 3050 0    60   Input ~ 0
 Ctrl
-Text HLabel 6350 2250 0    60   BiDi ~ 0
+Text HLabel 6350 2000 1    60   BiDi ~ 0
 A
-Text HLabel 6300 2400 0    60   BiDi ~ 0
+Text HLabel 6350 2600 3    60   BiDi ~ 0
 B
 $Comp
@@
 	5500 2600 5500 2800
 Wire Wire Line
-	5700 2600 5700 2500
+	5700 2600 5700 2450
 Connection ~ 5500 2600
 Wire Wire Line
-	5700 2000 5700 2100
+	5700 2000 5700 2150
 Connection ~ 5300 2000
 $Comp
@@
 Wire Wire Line
 	4800 2550 4800 2500
-Text Notes 5800 2300 0    60   ~ 0
-TODO
+$Comp
+L Relais_SPST REL?
+U 1 1 54E8CCF9
+P 5700 2300
+F 0 "REL?" H 5700 2500 60  0000 C CNN
+F 1 "Meder SIL05-1A72-71L" H 5700 2600 60  0000 C CNN
+F 2 "" H 5700 2300 60  0000 C CNN
+F 3 "" H 5700 2300 60  0000 C CNN
+	1    5700 2300
+	0    1    1    0
+$EndComp
+$Comp
+L Relais_SPST REL?
+U 2 1 54E8CD35
+P 6350 2300
+F 0 "REL?" H 6350 2500 60  0000 C CNN
+F 1 "Relais_SPST" H 6350 2000 60  0001 C CNN
+F 2 "" H 6350 2300 60  0000 C CNN
+F 3 "" H 6350 2300 60  0000 C CNN
+	2    6350 2300
+	0    1    1    0
+$EndComp
+Wire Wire Line
+	6350 2600 6350 2550
+Wire Wire Line
+	6350 2050 6350 2000
 $EndSCHEMATC

Commit message: Annotate schematic components
Parts:
- gave numbers to parts that had none: 8
Changed lines of the file:
@@
 B
 $Comp
-L BSS138 Q?
+L BSS138 Q9
 U 1 1 54E8DEE8
 P 5400 3000
-F 0 "Q?" H 5400 2851 40  0000 R CNN
+AR Path="/54D120FF/54E8DAE1/54E8DEE8" Ref="Q9"  Part="1"
+AR Path="/54D120FF/54E90580/54E8DEE8" Ref="Q10"  Part="1"
+F 0 "Q10" H 5400 2851 40  0000 R CNN
 F 1 "BSS138" H 5400 3150 40  0000 R CNN
 F 2 "SOT-23" H 5270 3102 29  0000 C CNN
@@
 $EndComp
 $Comp
-L R R?
+L R R50
 U 1 1 54E8DF2C
 P 5100 3400
-F 0 "R?" V 5180 3400 50  0000 C CNN
+AR Path="/54D120FF/54E8DAE1/54E8DF2C" Ref="R50"  Part="1"
+AR Path="/54D120FF/54E90580/54E8DF2C" Ref="R52"  Part="1"
+F 0 "R52" V 5180 3400 50  0000 C CNN
 F 1 "10k" V 5107 3401 50  0000 C CNN
 F 2 "" V 5030 3400 30  0000 C CNN
@@
 Connection ~ 5100 3050
 $Comp
-L GND #PWR?
+L GND #PWR133
 U 1 1 54E8DF95
 P 5100 3750
-F 0 "#PWR?" H 5100 3500 60  0001 C CNN
+AR Path="/54D120FF/54E8DAE1/54E8DF95" Ref="#PWR133"  Part="1"
+AR Path="/54D120FF/54E90580/54E8DF95" Ref="#PWR138"  Part="1"
+F 0 "#PWR138" H 5100 3500 60  0001 C CNN
 F 1 "GND" H 5100 3600 60  0000 C CNN
 F 2 "" H 5100 3750 60  0000 C CNN
@@
 	5100 3750 5100 3650
 $Comp
-L C C?
+L C C65
 U 1 1 54E8E18C
 P 4100 2300
-F 0 "C?" H 4150 2400 50  0000 L CNN
+AR Path="/54D120FF/54E8DAE1/54E8E18C" Ref="C65"  Part="1"
+AR Path="/54D120FF/54E90580/54E8E18C" Ref="C67"  Part="1"
+F 0 "C67" H 4150 2400 50  0000 L CNN
 F 1 "100n" H 4150 2200 50  0000 L CNN
 F 2 "" H 4138 2150 30  0000 C CNN
@@
 $EndComp
 $Comp
-L R R?
+L R R49
 U 1 1 54E8E1C0
 P 4450 2000
-F 0 "R?" V 4530 2000 50  0000 C CNN
+AR Path="/54D120FF/54E8DAE1/54E8E1C0" Ref="R49"  Part="1"
+AR Path="/54D120FF/54E90580/54E8E1C0" Ref="R51"  Part="1"
+F 0 "R51" V 4530 2000 50  0000 C CNN
 F 1 "180" V 4457 2001 50  0000 C CNN
 F 2 "" V 4380 2000 30  0000 C CNN
@@
 $EndComp
 $Comp
-L C C?
+L C C66
 U 1 1 54E8E27F
 P 4800 2300
-F 0 "C?" H 4850 2400 50  0000 L CNN
+AR Path="/54D120FF/54E8DAE1/54E8E27F" Ref="C66"  Part="1"
+AR Path="/54D120FF/54E90580/54E8E27F" Ref="C68"  Part="1"
+F 0 "C68" H 4850 2400 50  0000 L CNN
 F 1 "100n" H 4850 2200 50  0000 L CNN
 F 2 "" H 4838 2150 30  0000 C CNN
@@
 	4800 2000 4800 2100
 $Comp
-L GND #PWR?
+L GND #PWR131
 U 1 1 54E8E35E
 P 4100 2550
-F 0 "#PWR?" H 4100 2300 60  0001 C CNN
+AR Path="/54D120FF/54E8DAE1/54E8E35E" Ref="#PWR131"  Part="1"
+AR Path="/54D120FF/54E90580/54E8E35E" Ref="#PWR136"  Part="1"
+F 0 "#PWR136" H 4100 2300 60  0001 C CNN
 F 1 "GND" H 4100 2400 60  0000 C CNN
 F 2 "" H 4100 2550 60  0000 C CNN
@@
 	4800 2500 4800 2500
 $Comp
-L +9V #PWR?
+L +9V #PWR130
 U 1 1 54E8E5BD
 P 4000 1900
-F 0 "#PWR?" H 4000 1750 60  0001 C CNN
+AR Path="/54D120FF/54E8DAE1/54E8E5BD" Ref="#PWR130"  Part="1"
+AR Path="/54D120FF/54E90580/54E8E5BD" Ref="#PWR135"  Part="1"
+F 0 "#PWR135" H 4000 1750 60  0001 C CNN
 F 1 "+9V" H 4000 2040 60  0000 C CNN
 F 2 "" H 4000 1900 60  0000 C CNN
@@
 Connection ~ 4100 2000
 $Comp
-L GND #PWR?
+L GND #PWR134
 U 1 1 54E8E61E
 P 5500 3750
-F 0 "#PWR?" H 5500 3500 60  0001 C CNN
+AR Path="/54D120FF/54E8DAE1/54E8E61E" Ref="#PWR134"  Part="1"
+AR Path="/54D120FF/54E90580/54E8E61E" Ref="#PWR139"  Part="1"
+F 0 "#PWR139" H 5500 3500 60  0001 C CNN
 F 1 "GND" H 5500 3600 60  0000 C CNN
 F 2 "" H 5500 3750 60  0000 C CNN
@@
 	5500 3750 5500 3200
 $Comp
-L DIODE D?
+L DIODE D11
 U 1 1 54E8EB7A
 P 5300 2300
-F 0 "D?" H 5300 2400 50  0000 C CNN
+AR Path="/54D120FF/54E8DAE1/54E8EB7A" Ref="D11"  Part="1"
+AR Path="/54D120FF/54E90580/54E8EB7A" Ref="D12"  Part="1"
+F 0 "D12" H 5300 2400 50  0000 C CNN
 F 1 "DIODE" H 5300 2200 50  0000 C CNN
 F 2 "" H 5300 2300 60  0000 C CNN
@@
 Connection ~ 5300 2000
 $Comp
-L GND #PWR?
+L GND #PWR132
 U 1 1 54E8ED21
 P 4800 2550
-F 0 "#PWR?" H 4800 2300 60  0001 C CNN
+AR Path="/54D120FF/54E8DAE1/54E8ED21" Ref="#PWR132"  Part="1"
+AR Path="/54D120FF/54E90580/54E8ED21" Ref="#PWR137"  Part="1"
+F 0 "#PWR137" H 4800 2300 60  0001 C CNN
 F 1 "GND" H 4800 2400 60  0000 C CNN
 F 2 "" H 4800 2550 60  0000 C CNN
@@
 	4800 2550 4800 2500
 $Comp
-L Relais_SPST REL?
+L Relais_SPST REL9
 U 1 1 54E8CCF9
 P 5700 2300
-F 0 "REL?" H 5700 2500 60  0000 C CNN
+AR Path="/54D120FF/54E8DAE1/54E8CCF9" Ref="REL9"  Part="1"
+AR Path="/54D120FF/54E90580/54E8CCF9" Ref="REL11"  Part="1"
+F 0 "REL11" H 5700 2500 60  0000 C CNN
 F 1 "Meder SIL05-1A72-71L" H 5700 2600 60  0000 C CNN
 F 2 "" H 5700 2300 60  0000 C CNN
@@
 $EndComp
 $Comp
-L Relais_SPST REL?
+L Relais_SPST REL10
 U 2 1 54E8CD35
 P 6350 2300
-F 0 "REL?" H 6350 2500 60  0000 C CNN
+AR Path="/54D120FF/54E8DAE1/54E8CD35" Ref="REL10"  Part="2"
+AR Path="/54D120FF/54E90580/54E8CD35" Ref="REL12"  Part="2"
+F 0 "REL12" H 6350 2500 60  0000 C CNN
 F 1 "Relais_SPST" H 6350 2000 60  0001 C CNN
 F 2 "" H 6350 2300 60  0000 C CNN

Commit message: Set footprint of catch diode; Add datasheet
Parts:
- D11: footprint (none) -> Diodes_SMD:SOD-323
Changed lines of the file:
@@
 AR Path="/54D120FF/54E8DAE1/54E8DEE8" Ref="Q9"  Part="1"
 AR Path="/54D120FF/54E90580/54E8DEE8" Ref="Q10"  Part="1"
-F 0 "Q10" H 5400 2851 40  0000 R CNN
+F 0 "Q9" H 5400 2851 40  0000 R CNN
 F 1 "BSS138" H 5400 3150 40  0000 R CNN
 F 2 "SOT-23" H 5270 3102 29  0000 C CNN
@@
 AR Path="/54D120FF/54E8DAE1/54E8DF2C" Ref="R50"  Part="1"
 AR Path="/54D120FF/54E90580/54E8DF2C" Ref="R52"  Part="1"
-F 0 "R52" V 5180 3400 50  0000 C CNN
+F 0 "R50" V 5180 3400 50  0000 C CNN
 F 1 "10k" V 5107 3401 50  0000 C CNN
 F 2 "" V 5030 3400 30  0000 C CNN
@@
 AR Path="/54D120FF/54E8DAE1/54E8DF95" Ref="#PWR133"  Part="1"
 AR Path="/54D120FF/54E90580/54E8DF95" Ref="#PWR138"  Part="1"
-F 0 "#PWR138" H 5100 3500 60  0001 C CNN
+F 0 "#PWR133" H 5100 3500 60  0001 C CNN
 F 1 "GND" H 5100 3600 60  0000 C CNN
 F 2 "" H 5100 3750 60  0000 C CNN
@@
 AR Path="/54D120FF/54E8DAE1/54E8E18C" Ref="C65"  Part="1"
 AR Path="/54D120FF/54E90580/54E8E18C" Ref="C67"  Part="1"
-F 0 "C67" H 4150 2400 50  0000 L CNN
+F 0 "C65" H 4150 2400 50  0000 L CNN
 F 1 "100n" H 4150 2200 50  0000 L CNN
 F 2 "" H 4138 2150 30  0000 C CNN
@@
 AR Path="/54D120FF/54E8DAE1/54E8E1C0" Ref="R49"  Part="1"
 AR Path="/54D120FF/54E90580/54E8E1C0" Ref="R51"  Part="1"
-F 0 "R51" V 4530 2000 50  0000 C CNN
+F 0 "R49" V 4530 2000 50  0000 C CNN
 F 1 "180" V 4457 2001 50  0000 C CNN
 F 2 "" V 4380 2000 30  0000 C CNN
@@
 AR Path="/54D120FF/54E8DAE1/54E8E27F" Ref="C66"  Part="1"
 AR Path="/54D120FF/54E90580/54E8E27F" Ref="C68"  Part="1"
-F 0 "C68" H 4850 2400 50  0000 L CNN
+F 0 "C66" H 4850 2400 50  0000 L CNN
 F 1 "100n" H 4850 2200 50  0000 L CNN
 F 2 "" H 4838 2150 30  0000 C CNN
@@
 AR Path="/54D120FF/54E8DAE1/54E8E35E" Ref="#PWR131"  Part="1"
 AR Path="/54D120FF/54E90580/54E8E35E" Ref="#PWR136"  Part="1"
-F 0 "#PWR136" H 4100 2300 60  0001 C CNN
+F 0 "#PWR131" H 4100 2300 60  0001 C CNN
 F 1 "GND" H 4100 2400 60  0000 C CNN
 F 2 "" H 4100 2550 60  0000 C CNN
@@
 AR Path="/54D120FF/54E8DAE1/54E8E5BD" Ref="#PWR130"  Part="1"
 AR Path="/54D120FF/54E90580/54E8E5BD" Ref="#PWR135"  Part="1"
-F 0 "#PWR135" H 4000 1750 60  0001 C CNN
+F 0 "#PWR130" H 4000 1750 60  0001 C CNN
 F 1 "+9V" H 4000 2040 60  0000 C CNN
 F 2 "" H 4000 1900 60  0000 C CNN
@@
 AR Path="/54D120FF/54E8DAE1/54E8E61E" Ref="#PWR134"  Part="1"
 AR Path="/54D120FF/54E90580/54E8E61E" Ref="#PWR139"  Part="1"
-F 0 "#PWR139" H 5500 3500 60  0001 C CNN
+F 0 "#PWR134" H 5500 3500 60  0001 C CNN
 F 1 "GND" H 5500 3600 60  0000 C CNN
 F 2 "" H 5500 3750 60  0000 C CNN
@@
 AR Path="/54D120FF/54E8DAE1/54E8EB7A" Ref="D11"  Part="1"
 AR Path="/54D120FF/54E90580/54E8EB7A" Ref="D12"  Part="1"
-F 0 "D12" H 5300 2400 50  0000 C CNN
+F 0 "D11" H 5300 2400 50  0000 C CNN
 F 1 "DIODE" H 5300 2200 50  0000 C CNN
-F 2 "" H 5300 2300 60  0000 C CNN
+F 2 "Diodes_SMD:SOD-323" H 5300 2300 60  0001 C CNN
 F 3 "" H 5300 2300 60  0000 C CNN
 	1    5300 2300
@@
 AR Path="/54D120FF/54E8DAE1/54E8ED21" Ref="#PWR132"  Part="1"
 AR Path="/54D120FF/54E90580/54E8ED21" Ref="#PWR137"  Part="1"
-F 0 "#PWR137" H 4800 2300 60  0001 C CNN
+F 0 "#PWR132" H 4800 2300 60  0001 C CNN
 F 1 "GND" H 4800 2400 60  0000 C CNN
 F 2 "" H 4800 2550 60  0000 C CNN
@@
 AR Path="/54D120FF/54E8DAE1/54E8CCF9" Ref="REL9"  Part="1"
 AR Path="/54D120FF/54E90580/54E8CCF9" Ref="REL11"  Part="1"
-F 0 "REL11" H 5700 2500 60  0000 C CNN
+F 0 "REL9" H 5700 2500 60  0000 C CNN
 F 1 "Meder SIL05-1A72-71L" H 5700 2600 60  0000 C CNN
 F 2 "" H 5700 2300 60  0000 C CNN
@@
 AR Path="/54D120FF/54E8DAE1/54E8CD35" Ref="REL10"  Part="2"
 AR Path="/54D120FF/54E90580/54E8CD35" Ref="REL12"  Part="2"
-F 0 "REL12" H 6350 2500 60  0000 C CNN
+F 0 "REL10" H 6350 2500 60  0000 C CNN
 F 1 "Relais_SPST" H 6350 2000 60  0001 C CNN
 F 2 "" H 6350 2300 60  0000 C CNN
