File: hardware/vca.sch (KiCad schematic (older format))
At the start: 0 parts

Commit message: Stub VCA schematic sheet
Parts:
- added U?: THAT2180, symbol THAT2180
Changed lines of the file:
@@
 $Descr A4 11693 8268
 encoding utf-8
-Sheet 2 23
+Sheet 23 23
 Title ""
 Date ""
@@
 Comment4 ""
 $EndDescr
+$Comp
+L THAT2180 U?
+U 1 1 54EA31E2
+P 5600 3700
+F 0 "U?" H 5900 4050 60  0000 C CNN
+F 1 "THAT2180" H 6000 3900 60  0000 C CNN
+F 2 "" H 5600 3700 60  0000 C CNN
+F 3 "" H 5600 3700 60  0000 C CNN
+	1    5600 3700
+	1    0    0    -1
+$EndComp
 $EndSCHEMATC
