File: hardware/wah.sch (KiCad schematic (older format))
At the start: 21 parts

Commit message: Annotate schematic components
Parts:
- removed C?: 10u, symbol C
- added C40: 10u, symbol C
- gave numbers to parts that had none: 20
Connections:
- net 9V_Wah: now also C40.2
- net GND: now also C40.1
Changed lines of the file:
@@
 9V_Wah
 $Comp
-L R R?
+L R R1
 U 1 1 54D5397B
 P 3650 2300
-F 0 "R?" V 3730 2300 50  0000 C CNN
+F 0 "R1" V 3730 2300 50  0000 C CNN
 F 1 "100k" V 3657 2301 50  0000 C CNN
 F 2 "" V 3580 2300 30  0000 C CNN
@@
 $EndComp
 $Comp
-L C C?
+L C C42
 U 1 1 54D53A9D
 P 4350 2050
-F 0 "C?" H 4400 2150 50  0000 L CNN
+F 0 "C42" H 4400 2150 50  0000 L CNN
 F 1 "1n" H 4400 1950 50  0000 L CNN
 F 2 "" H 4388 1900 30  0000 C CNN
@@
 $EndComp
 $Comp
-L R R?
+L R R2
 U 1 1 54D53B3B
 P 4350 2300
-F 0 "R?" V 4430 2300 50  0000 C CNN
+F 0 "R2" V 4430 2300 50  0000 C CNN
 F 1 "82k" V 4357 2301 50  0000 C CNN
 F 2 "" V 4280 2300 30  0000 C CNN
@@
 $EndComp
 $Comp
-L C C?
+L C C43
 U 1 1 54D53C29
 P 5000 2300
-F 0 "C?" H 5050 2400 50  0000 L CNN
+F 0 "C43" H 5050 2400 50  0000 L CNN
 F 1 "47n" H 5050 2200 50  0000 L CNN
 F 2 "" H 5038 2150 30  0000 C CNN
@@
 $EndComp
 $Comp
-L LM741 U?
+L LM741 U10
 U 1 1 54D53DF6
 P 6000 2200
-F 0 "U?" H 6150 2350 60  0000 C CNN
+F 0 "U10" H 6150 2350 60  0000 C CNN
 F 1 "LM741" H 6150 2450 60  0000 C CNN
 F 2 "" H 6000 2200 60  0000 C CNN
@@
 $EndComp
 $Comp
-L GND #PWR?
+L GND #PWR64
 U 1 1 54D53F40
 P 2650 1650
-F 0 "#PWR?" H 2650 1400 60  0001 C CNN
+F 0 "#PWR64" H 2650 1400 60  0001 C CNN
 F 1 "GND" H 2650 1500 60  0001 C CNN
 F 2 "" H 2650 1650 60  0000 C CNN
@@
 $EndComp
 $Comp
-L GND #PWR?
+L GND #PWR68
 U 1 1 54D540D2
 P 5900 2600
-F 0 "#PWR?" H 5900 2350 60  0001 C CNN
+F 0 "#PWR68" H 5900 2350 60  0001 C CNN
 F 1 "GND" H 5900 2450 60  0001 C CNN
 F 2 "" H 5900 2600 60  0000 C CNN
@@
 $EndComp
 $Comp
-L R R?
+L R R3
 U 1 1 54D54136
 P 4450 1000
-F 0 "R?" V 4530 1000 50  0000 C CNN
+F 0 "R3" V 4530 1000 50  0000 C CNN
 F 1 "100k" V 4457 1001 50  0000 C CNN
 F 2 "" V 4380 1000 30  0000 C CNN
@@
 $EndComp
 $Comp
-L R R?
+L R R4
 U 1 1 54D54235
 P 4800 1350
-F 0 "R?" V 4880 1350 50  0000 C CNN
+F 0 "R4" V 4880 1350 50  0000 C CNN
 F 1 "100k" V 4807 1351 50  0000 C CNN
 F 2 "" V 4730 1350 30  0000 C CNN
@@
 $EndComp
 $Comp
-L C C?
+L C C44
 U 1 1 54D542A6
 P 5100 1350
-F 0 "C?" H 5150 1450 50  0000 L CNN
+F 0 "C44" H 5150 1450 50  0000 L CNN
 F 1 "10u" H 5150 1250 50  0000 L CNN
 F 2 "" H 5138 1200 30  0000 C CNN
@@
 $EndComp
 $Comp
-L GND #PWR?
+L GND #PWR66
 U 1 1 54D54455
 P 4800 1600
-F 0 "#PWR?" H 4800 1350 60  0001 C CNN
+F 0 "#PWR66" H 4800 1350 60  0001 C CNN
 F 1 "GND" H 4800 1450 60  0001 C CNN
 F 2 "" H 4800 1600 60  0000 C CNN
@@
 $EndComp
 $Comp
-L GND #PWR?
+L GND #PWR67
 U 1 1 54D54478
 P 5100 1600
-F 0 "#PWR?" H 5100 1350 60  0001 C CNN
+F 0 "#PWR67" H 5100 1350 60  0001 C CNN
 F 1 "GND" H 5100 1450 60  0001 C CNN
 F 2 "" H 5100 1600 60  0000 C CNN
@@
 $EndComp
 $Comp
-L C C?
-U 1 1 54D54B27
+L C C40
+U 1 1 54E9CACA
 P 2500 1300
-F 0 "C?" H 2550 1400 50  0000 L CNN
+F 0 "C40" H 2550 1400 50  0000 L CNN
 F 1 "10u" H 2550 1200 50  0000 L CNN
 F 2 "" H 2538 1150 30  0000 C CNN
@@
 $EndComp
 $Comp
-L C C?
+L C C41
 U 1 1 54D54B9A
 P 2800 1300
-F 0 "C?" H 2850 1400 50  0000 L CNN
+F 0 "C41" H 2850 1400 50  0000 L CNN
 F 1 "10u" H 2850 1200 50  0000 L CNN
 F 2 "" H 2838 1150 30  0000 C CNN
@@
 9V_Wah
 $Comp
-L C C?
+L C C46
 U 1 1 54D554E3
 P 5800 2850
-F 0 "C?" H 5850 2950 50  0000 L CNN
+F 0 "C46" H 5850 2950 50  0000 L CNN
 F 1 "5p" H 5850 2750 50  0000 L CNN
 F 2 "" H 5838 2700 30  0000 C CNN
@@
 $EndComp
 $Comp
-L R R?
+L R R7
 U 1 1 54D55528
 P 6300 2850
-F 0 "R?" V 6380 2850 50  0000 C CNN
+F 0 "R7" V 6380 2850 50  0000 C CNN
 F 1 "1.2M" V 6307 2851 50  0000 C CNN
 F 2 "" V 6230 2850 30  0000 C CNN
@@
 $EndComp
 $Comp
-L R R?
+L R R6
 U 1 1 54D555D7
 P 6050 3100
-F 0 "R?" V 6130 3100 50  0000 C CNN
+F 0 "R6" V 6130 3100 50  0000 C CNN
 F 1 "470k" V 6057 3101 50  0000 C CNN
 F 2 "" V 5980 3100 30  0000 C CNN
@@
 $EndComp
 $Comp
-L C C?
+L C C45
 U 1 1 54D55B50
 P 5350 3400
-F 0 "C?" H 5400 3500 50  0000 L CNN
+F 0 "C45" H 5400 3500 50  0000 L CNN
 F 1 "6.8n" H 5400 3300 50  0000 L CNN
 F 2 "" H 5388 3250 30  0000 C CNN
@@
 $EndComp
 $Comp
-L C C?
+L C C47
 U 1 1 54D55BC2
 P 6650 3400
-F 0 "C?" H 6700 3500 50  0000 L CNN
+F 0 "C47" H 6700 3500 50  0000 L CNN
 F 1 "2n" H 6700 3300 50  0000 L CNN
 F 2 "" H 6688 3250 30  0000 C CNN
@@
 $EndComp
 $Comp
-L C C?
+L C C48
 U 1 1 54D563C0
 P 7000 2200
-F 0 "C?" H 7050 2300 50  0000 L CNN
+F 0 "C48" H 7050 2300 50  0000 L CNN
 F 1 "1u" H 7050 2100 50  0000 L CNN
 F 2 "" H 7038 2050 30  0000 C CNN
@@
 $EndComp
 $Comp
-L POT RV?
+L POT RV1
 U 1 1 54D56709
 P 7350 2600
-F 0 "RV?" H 7350 2500 50  0000 C CNN
+F 0 "RV1" H 7350 2500 50  0000 C CNN
 F 1 "10k" H 7350 2600 50  0000 C CNN
 F 2 "" H 7350 2600 60  0000 C CNN
@@
 $EndComp
 $Comp
-L GND #PWR?
+L GND #PWR71
 U 1 1 54D56848
 P 7350 2950
-F 0 "#PWR?" H 7350 2700 60  0001 C CNN
+F 0 "#PWR71" H 7350 2700 60  0001 C CNN
 F 1 "GND" H 7350 2800 60  0001 C CNN
 F 2 "" H 7350 2950 60  0000 C CNN
@@
 	2500 1600 2800 1600
 $Comp
-L Jack_Stacked CON?
+L Jack_Stacked CON9
 U 1 1 54E8B32C
 P 4600 7300
-F 0 "CON?" H 3750 9300 60  0000 C CNN
+F 0 "CON9" H 3750 9300 60  0000 C CNN
 F 1 "Jack_Stacked" H 3700 7550 60  0000 C CNN
 F 2 "" H 4600 7300 60  0000 C CNN
@@
 Wah Input
 $Comp
-L GNDA #PWR?
+L GNDA #PWR65
 U 1 1 54E8E591
 P 3050 7350
-F 0 "#PWR?" H 3050 7100 60  0001 C CNN
+F 0 "#PWR65" H 3050 7100 60  0001 C CNN
 F 1 "GNDA" H 3050 7200 60  0000 C CNN
 F 2 "" H 3050 7350 60  0000 C CNN
@@
 Connection ~ 3050 6850
 $Comp
-L Photores R?
+L Photores R5
 U 1 1 54E8FBBB
 P 6000 5050
-F 0 "R?" V 6080 5050 50  0000 C CNN
+F 0 "R5" V 6080 5050 50  0000 C CNN
 F 1 "Photores" V 6210 5050 50  0000 C TNN
 F 2 "" V 5930 5050 30  0000 C CNN
@@
 $EndComp
 $Comp
-L GND #PWR?
+L GND #PWR69
 U 1 1 54E8FD73
 P 6000 5350
-F 0 "#PWR?" H 6000 5100 60  0001 C CNN
+F 0 "#PWR69" H 6000 5100 60  0001 C CNN
 F 1 "GND" H 6000 5200 60  0001 C CNN
 F 2 "" H 6000 5350 60  0000 C CNN
@@
 	6000 5350 6000 5300
 $Comp
-L LED D?
+L LED D2
 U 1 1 54E90184
 P 6550 5050
-F 0 "D?" H 6550 5150 50  0000 C CNN
+F 0 "D2" H 6550 5150 50  0000 C CNN
 F 1 "LED" H 6550 4950 50  0000 C CNN
 F 2 "" H 6550 5050 60  0000 C CNN
@@
 $EndComp
 $Comp
-L GND #PWR?
+L GND #PWR70
 U 1 1 54E902B7
 P 6550 5350
-F 0 "#PWR?" H 6550 5100 60  0001 C CNN
+F 0 "#PWR70" H 6550 5100 60  0001 C CNN
 F 1 "GND" H 6550 5200 60  0001 C CNN
 F 2 "" H 6550 5350 60  0000 C CNN
@@
 	6550 5350 6550 5250
 $Comp
-L R R?
+L R R8
 U 1 1 54E906C6
 P 6950 4700
-F 0 "R?" V 7030 4700 50  0000 C CNN
+F 0 "R8" V 7030 4700 50  0000 C CNN
 F 1 "R" V 6957 4701 50  0000 C CNN
 F 2 "" V 6880 4700 30  0000 C CNN
